File: hw/pnc_probe.sch (EAGLE design)
At the start: 14 parts, among them U1 TPS6024X_VSSOP8, U2 DUAL_NAND_SSOP8, U3 MF-DSC-SOT233-BSS138, X1 0446200002, X2 0446200002

Commit message: Fix r1 errata
* The footprint for the TPS6024 was wrong.  I wasn't able to find a
  sample one, so used a generic VSSOP originally, but that didn't
  match the TI part.  I instead used rough dimensions from a KiCAD
  model and double checked against the datasheet.
* Yikes, I had left some airwires!
* Added test points for gnd, power, and the final probe signal.
Parts:
- added 3V3, 5V, GND, PRB: (no value), pinhead:PINHD-1X1
Connections:
- net GND: now also GND.1
- net PROBE: now also PRB.1
- net VCC_3V: now also 3V3.1
- net VCC_5V: now also 5V.1
Other:
- note added: "Pocket NC - vers.by - Touch Probe Adapter r2 (c) 2021 Josh Pieper - jjp@pobox.com Available under the Apache 2.0 License"
- note removed: "Pocket NC - vers.by - Touch Probe Adapter (c) 2021 Josh Pieper - jjp@pobox.com Available under the Apache 2.0 License"
Changed lines of the file:
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@@
 </part>
 <part name="GND9" library="supply1" library_urn="urn:adsk.eagle:library:371" deviceset="GND" device=""/>
+<part name="GND" library="pinhead" library_urn="urn:adsk.eagle:library:325" deviceset="PINHD-1X1" device="" package3d_urn="urn:adsk.eagle:package:22485/2"/>
+<part name="3V3" library="pinhead" library_urn="urn:adsk.eagle:library:325" deviceset="PINHD-1X1" device="" package3d_urn="urn:adsk.eagle:package:22485/2"/>
+<part name="5V" library="pinhead" library_urn="urn:adsk.eagle:library:325" deviceset="PINHD-1X1" device="" package3d_urn="urn:adsk.eagle:package:22485/2"/>
+<part name="PRB" library="pinhead" library_urn="urn:adsk.eagle:library:325" deviceset="PINHD-1X1" device="" package3d_urn="urn:adsk.eagle:package:22485/2"/>
+<part name="GND10" library="supply1" library_urn="urn:adsk.eagle:library:371" deviceset="GND" device=""/>
 </parts>
 <sheets>
@@
 <text x="81.28" y="81.28" size="1.778" layer="91">1/2 = motor phase 1
 3/4 = motor phase 2</text>
-<text x="-17.78" y="96.52" size="1.778" layer="97">Pocket NC - vers.by - Touch Probe Adapter
+<text x="-17.78" y="96.52" size="1.778" layer="97">Pocket NC - vers.by - Touch Probe Adapter r2
 (c) 2021 Josh Pieper - jjp@pobox.com
 Available under the Apache 2.0 License</text>
@@
 <instance part="GND9" gate="1" x="99.06" y="-86.36" smashed="yes">
 <attribute name="VALUE" x="96.52" y="-88.9" size="1.778" layer="96"/>
+</instance>
+<instance part="GND" gate="G$1" x="157.48" y="-60.96" smashed="yes">
+<attribute name="NAME" x="151.13" y="-57.785" size="1.778" layer="95"/>
+<attribute name="VALUE" x="151.13" y="-66.04" size="1.778" layer="96"/>
+</instance>
+<instance part="3V3" gate="G$1" x="157.48" y="-68.58" smashed="yes">
+<attribute name="NAME" x="151.13" y="-65.405" size="1.778" layer="95"/>
+<attribute name="VALUE" x="151.13" y="-73.66" size="1.778" layer="96"/>
+</instance>
+<instance part="5V" gate="G$1" x="157.48" y="-76.2" smashed="yes">
+<attribute name="NAME" x="151.13" y="-73.025" size="1.778" layer="95"/>
+<attribute name="VALUE" x="151.13" y="-81.28" size="1.778" layer="96"/>
+</instance>
+<instance part="PRB" gate="G$1" x="157.48" y="-83.82" smashed="yes">
+<attribute name="NAME" x="151.13" y="-80.645" size="1.778" layer="95"/>
+<attribute name="VALUE" x="151.13" y="-88.9" size="1.778" layer="96"/>
+</instance>
+<instance part="GND10" gate="1" x="137.16" y="-63.5" smashed="yes">
+<attribute name="VALUE" x="134.62" y="-66.04" size="1.778" layer="96"/>
 </instance>
 </instances>
@@
 <pinref part="GND9" gate="1" pin="GND"/>
 </segment>
+<segment>
+<pinref part="GND" gate="G$1" pin="1"/>
+<wire x1="154.94" y1="-60.96" x2="137.16" y2="-60.96" width="0.1524" layer="91"/>
+<pinref part="GND10" gate="1" pin="GND"/>
+</segment>
 </net>
 <net name="PROBE" class="0">
@@
 <wire x1="180.34" y1="12.7" x2="180.34" y2="35.56" width="0.1524" layer="91"/>
 <label x="185.42" y="33.02" size="1.778" layer="95"/>
+</segment>
+<segment>
+<pinref part="PRB" gate="G$1" pin="1"/>
+<wire x1="154.94" y1="-83.82" x2="137.16" y2="-83.82" width="0.1524" layer="91"/>
+<label x="139.7" y="-83.82" size="1.778" layer="95"/>
 </segment>
 </net>
@@
 <junction x="22.86" y="-60.96"/>
 </segment>
+<segment>
+<pinref part="3V3" gate="G$1" pin="1"/>
+<wire x1="154.94" y1="-68.58" x2="137.16" y2="-68.58" width="0.1524" layer="91"/>
+<label x="139.7" y="-68.58" size="1.778" layer="95"/>
+</segment>
 </net>
 <net name="VCC_5V" class="0">
@@
 <junction x="99.06" y="-60.96"/>
 </segment>
-</net>
+<segment>
+<pinref part="5V" gate="G$1" pin="1"/>
+<wire x1="154.94" y1="-76.2" x2="137.16" y2="-76.2" width="0.1524" layer="91"/>
+<label x="139.7" y="-76.2" size="1.778" layer="95"/>
+</segment>
+</net>

Commit message: Fix a component value
Parts:
- R3: MPN MF-RES-0603-100K -> MF-RES-0603-4.7K
Changed lines of the file:
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@@
 <part name="R3" library="mfpassives" deviceset="RESISTOR" device="_0603" value="4.7k">
 <attribute name="HOUSEPART" value="YES"/>
-<attribute name="MPN" value="MF-RES-0603-100K"/>
+<attribute name="MPN" value="MF-RES-0603-4.7K"/>
 </part>
 <part name="U1" library="pnc_probe" deviceset="TPS6024X" device="_VSSOP8"/>
